File: tida-050047-ledcontroller.kicad_sch (KiCad schematic)
At the start: 83 parts, among them U1 TPS25750DRJKR, U2 CAT24C256WI-GT3, U3 TLV75533PDBVR, U4 TPS54531DDAR, U5 BQ25798RQMR

Commit message: update from fiver
Parts:
- removed C10, C11, C12, C13: 0.01uF, Capacitor_SMD:C_0603_1608Metric_Pad1.08x0.95mm_HandSolder, symbol Device:C
- removed C14: 4.7uF, Capacitor_SMD:C_0805_2012Metric_Pad1.18x1.45mm_HandSolder, symbol Device:C
- removed C19: CA45-B-6.3V-100UF-K, easyeda2kicad:CAP-SMD_L3.5-W2.8-R-RD, symbol easyeda2kicad:CA45-B-6.3V-100UF-K
- removed D1: TVS2200DRVR, easyeda2kicad:WSON-6_L2.0-W2.0-P0.65-BL-EP, symbol easyeda2kicad:TVS2200DRVR
- removed D2: SS54_C123946, easyeda2kicad:SMA_L4.4-W2.8-LS5.4-RD, symbol easyeda2kicad:SS54_C123946
- removed F1: BSMD2920-600-16V, easyeda2kicad:F2920, symbol easyeda2kicad:BSMD2920-600-16V
- removed FB1: FerriteBead, Resistor_SMD:R_0805_2012Metric_Pad1.20x1.40mm_HandSolder, symbol Device:FerriteBead
- removed L1: GCDA0650-4R7MC, easyeda2kicad:IND-SMD_L7.6-W6.6, symbol easyeda2kicad:GCDA0650-4R7MC
- removed L2: CYA0630-1.0UH, easyeda2kicad:IND-SMD_L7.2-W6.6_GPSR0730, symbol easyeda2kicad:CYA0630-1.0UH
- added BT1, BT2, BT3, BT4: BH-18650-B1BA002, easyeda2kicad:BATTERY-SMD_18650-1S-L77.1-W20.7-1, symbol easyeda2kicad:BH-18650-B1BA002
- added C19, C51, C52, C53: 100nF, symbol Device:C_Polarized
- added C50: 100uF/6.3V, symbol Device:C_Polarized
- added C54: 4.7uF, Capacitor_SMD:C_0805_2012Metric_Pad1.18x1.45mm_HandSolder, symbol Device:C
- added C55, C56, C57, C58: 0.01uF, Capacitor_SMD:C_0603_1608Metric_Pad1.08x0.95mm_HandSolder, symbol Device:C
- added D2: TVS2200DRVR, easyeda2kicad:WSON-6_L2.0-W2.0-P0.65-BL-EP, symbol easyeda2kicad:TVS2200DRVR
- added D3: CDBC540-G, Diode_SMD:D_SMC, symbol Diode:CDBA340-HF
- added F2: BSMD2920-600-16V, easyeda2kicad:F2920, symbol easyeda2kicad:BSMD2920-600-16V
- added H4: PZ254V-11-02P, easyeda2kicad:HDR-TH_2P-P2.54-V-M, symbol easyeda2kicad:PZ254V-11-02P
- added JP1, JP2, JP3, JP4, JP5, JP6: SolderJumper_2_Bridged, symbol Jumper:SolderJumper_2_Bridged
- added L1: 4.7uH, symbol Device:L_Iron
- added L2: 1uH, symbol Device:L_Iron
- added Q3, Q4, Q5, Q6: BSL802SN, symbol Simulation_SPICE:NMOS
- added R19, R22, R25, R28: 100R, Resistor_SMD:R_0603_1608Metric_Pad0.98x0.95mm_HandSolder, symbol Device:R
- added R20, R21, R23, R24, R26, R27, R29, R30: 20R, Resistor_SMD:R_0603_1608Metric_Pad0.98x0.95mm_HandSolder, symbol Device:R
- added U10: XT30PW-F, easyeda2kicad:CONN-TH_XT30PW-F-1, symbol easyeda2kicad:XT30PW-F
- added U11, U7, U8, U9: HY2213-BB3A, easyeda2kicad:SOT-23-6_L2.9-W1.6-P0.95-LS2.8-BR, symbol easyeda2kicad:HY2213-BB3A
- C15, C16: value 4.7uF -> 4.7uF/50V
- C20: value 10nF -> 10nF/50V
- C21: value 10nF -> 10nF/100V
- C23: value 10nF -> 2.2nF/100V
- C24: value 22pF -> 22pF/50V
- C34, C35: now not fitted
- C36: value 4.7uF -> 4.7uF/25V
- C37, C38: value 0.1uF -> 0.047uF
- C39: value 0.1uF -> 1000pF/50V
- C41: value 0.1uF -> 0.1uF/50V
- C43, C44, C45, C46: value 10uF -> 10uF/25V
Connections:
- net AGND: now also C39.1, NT1.1
- net BATT: now also BT4.2, JP4.2 (B), R29.1, R30.1
- net GND: now also C17.2, C18.2, R11.1, BT1.1, C19.2, C50.2, C54.1, C55.1, C56.1, C57.1, C58.1, D2.1 (GND), D2.2 (GND), D2.3 (GND), D2.7 (GND), D3.2 (A), H4.1, Q3.3 (S), U10.2, U11.3 (VSS)
- net I2C_SCL: now also JP5.1 (A); no longer U5.14 (SCL)
- net I2C_SDA: now also JP6.1 (A); no longer U5.15 (SDA)
- net PP5V: now also C50.1, L1.2, U10.1
- net SYS: now also H4.2
- net VBUS: now also F2.2
- net at USB1.A4B9 (VBUS), USB1.B4A9 (VBUS): now also C54.2, C55.2, C56.2, C57.2, C58.2, D2.4 (IN), D2.5 (IN), D2.6 (IN), F2.1
- net at C37.1, U5.28 (SW1): now also L2.1
- net at U5.26 (SW2): now also C38.2, L2.2; no longer C38.1
- net at C22.2, U4.8 (PH): now also D3.1 (K), L1.1
- net at U5.19 (BTST2): now also C38.1; no longer C38.2
- new net: JP6.2 (B), U5.15 (SDA)
- new net: C19.1, R19.2, U11.2 (VDD)
- new net: Q3.2 (G), U11.6 (OUT)
- new net: C53.1, R28.2, U9.2 (VDD)
- new net: Q6.1 (D), R29.2, R30.2
- new net: Q5.1 (D), R26.2, R27.2
- new net: JP3.1 (A), R22.1
- new net: C51.1, R22.2, U7.2 (VDD)
- new net: Q4.2 (G), U7.6 (OUT)
- new net: JP1.1 (A), R19.1
- new net: Q6.2 (G), U9.6 (OUT)
- new net: JP5.2 (B), U5.14 (SCL)
- new net: JP2.1 (A), R25.1
- new net: Q3.1 (D), R20.2, R21.2
- new net: Q4.1 (D), R23.2, R24.2
- new net: C52.1, R25.2, U8.2 (VDD)
- new net: JP4.1 (A), R28.1
- new net: Q5.2 (G), U8.6 (OUT)
- new net BATT1 OUT+: BT1.2, BT2.1, C52.2, JP1.2 (B), Q5.3 (S), R20.1, R21.1, U8.3 (VSS)
- new net BATT2 OUT+: BT2.2, BT3.1, C51.2, JP2.2 (B), Q4.3 (S), R26.1, R27.1, U7.3 (VSS)
- new net BATT3 OUT+: BT3.2, BT4.1, C53.2, JP3.2 (B), Q6.3 (S), R23.1, R24.1, U9.3 (VSS)
Other:
- note added: "Cell Balancing Circuit"
- note added: "Power 5V TO 3.3V"
- note added: "USB-C WITH FUSE,NOISE AND ESD PROTECTION"
- note added: "XT30PW-F Connector Output to other board"
- note removed: "DC/DC power design"
- note removed: "USB-C with Fuse, Noise and ESD Protection"
- moved on the sheet: C1, C15, C16, C17, C18, C2, C20, C21, C22, C23, C24, C25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
